File: hardware/kicad/power.kicad_sch (KiCad schematic)
At the start: 61 parts, among them J1 USB_C_Receptacle_USB2.0_16P, J2 BATT (1S LiPo), U1 BQ24073RGT, U2 TPS63802DLA, U3 TPS61023DRL, U4 TPS22965DSG, U5 USBLC6-2SC6, U6 TPS63900DSK, U7 MCP1700T-3002E/TT

Commit message: Schematic: Power sheet redrawn with wired circuits; docs
Power (now A2): VBUS rail across the top from USB-C through the charger
input with C1, R20 and a PWR_FLAG on it; CC pull-downs inline; D+/D- run
straight to the MCU labels with the USBLC6 tapped on; BQ24073 straps on a
GND rail, TS/NTC/filter, CHG LED chain, OUT/BAT caps wired; RTC LDO,
battery divider, TPS63802/TPS61023 with input rails, bridged inductors,
feedback dividers and output banks; load switch with the R13 bypass drawn
across it; reserved TPS63900 block likewise. Local nets whose names are
checked or used by net classes keep labels on their wires.
Electrically identical (156 parts, 193 nets); board re-synced: DRC 0
unconnected / 0 parity, ERC 0. README/TODO: scripts are the schematic's
source of truth; compare_netlists / sync_board_to_schematic documented.

Co-Authored-By: Claude Opus 5.5 <noreply@anthropic.com>
Parts:
- removed RT1: 10k NTC, Connector_Wire:SolderWire-0.1sqmm_1x02_P3.6mm_D0.4mm_OD1mm, symbol Device:Thermistor_NTC
- removed TP6: GND, TestPoint:TestPoint_Pad_D1.5mm, symbol Connector:TestPoint
- removed U2: TPS63802DLA, epaper:Texas_DLA0010A_VSON-HR-10_2x3mm_P0.5mm, symbol epaper:TPS63802
- added C18: 100nF, Capacitor_SMD:C_0402_1005Metric, symbol Device:C
- added L1: 0.47uH, Inductor_SMD:L_Murata_DFE201610P, symbol Device:L
- added R13: 0R, Resistor_SMD:R_0603_1608Metric, symbol Device:R
- RT1: renamed from C18; value 100nF -> 10k NTC; footprint Capacitor_SMD:C_0402_1005Metric -> Connector_Wire:SolderWire-0.1sqmm_1x02_P3.6mm_D0.4mm_OD1mm; symbol Device:C -> Device:Thermistor_NTC; MPN (none) -> NXFT15XH103FA2B (Murata leaded film NTC: same 10k/B=3380 cu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
- TP6: renamed from R13; value 0R -> GND; footprint Resistor_SMD:R_0603_1608Metric -> TestPoint:TestPoint_Pad_D1.5mm; symbol Device:R -> Connector:TestPoint; now fitted
- U2: renamed from L1; value 0.47uH -> TPS63802DLA; footprint Inductor_SMD:L_Murata_DFE201610P -> epaper:Texas_DLA0010A_VSON-HR-10_2x3mm_P0.5mm; symbol Device:L -> epaper:TPS63802; MPN DFE201612E-R47M=P2 (Isat 5.5A, 26mR; Murata land = this foo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 -> TPS63802DLAR
Connections:
- net +3V3: now also U2.6 (VOUT), R13.1; no longer TP6.1
- net 3V3_PERIPH: now also R13.2; no longer TP6.2
- net 3V3_PG: now also U2.5 (PG)
- net BB_EN: now also U2.1 (EN)
- net BB_FB: now also U2.4 (FB)
- net BB_L1: now also U2.9 (L1), L1.1; no longer U2.1
- net BB_L2: now also U2.7 (L2), L1.2; no longer U2.2
- net GND: now also TP6.1, U2.2 (MODE), U2.3 (AGND), U2.8 (GND), C18.2
- net TS: now also RT1.1
- net TS_SENSE: now also C18.1; no longer RT1.1
- net VSYS: now also U2.10 (VIN)
Other:
- note added: "POWER — USB-C in, LiPo charger + power path, 3V3 buck-boost, 5V boost, RTC backup, peripheral load switch, reserved always-on rail. Generated by hardware/scripts/gen_schematic.py (sheet_power.py)."
- note removed: "POWER — draft (generated by hardware/scripts/gen_schematic.py; edit in Eeschema from here on) See README.md "Custom PCB (Planned)" and TODO.md for the open questions on this sheet."
- moved on the sheet: U1
